File: PreAmp/ClassD.kicad_sch (KiCad schematic)
At the start: 42 parts, among them J1 Conn_01x02_Pin, J2 Conn_01x02_Pin, J3 Conn_01x03, U1 L78L09_TO92, U2 LM358, U3 TL494

Commit message: Init Full Bridge Topology
Parts:
- removed J2: Conn_01x02_Pin, Connector_JST:JST_XH_B2B-XH-A_1x02_P2.50mm_Vertical, symbol Connector:Conn_01x02_Pin
- added C11: C_Small, Capacitor_THT:C_Disc_D5.0mm_W2.5mm_P5.00mm, symbol Device:C_Small
- added C12: C_Small_US, Capacitor_THT:CP_Radial_D5.0mm_P2.00mm, symbol Device:C_Small_US
- added C13, C14: C_Small, Capacitor_THT:C_Disc_D3.8mm_W2.6mm_P2.50mm, symbol Device:C_Small
- added C15: 100uF, Capacitor_THT:CP_Radial_D8.0mm_P3.50mm, symbol Device:C_Polarized_Small
- added C5: C_Polarized_Small, Capacitor_THT:CP_Radial_D5.0mm_P2.00mm, symbol Device:C_Polarized_Small
- added J2: AudioJack3, symbol Connector_Audio:AudioJack3
- added J4: Conn_01x03, Connector_JST:JST_XH_B3B-XH-A_1x03_P2.50mm_Vertical, symbol Connector_Generic:Conn_01x03
- added R13, R14, R15, R16, R17, R18, R19, R20: R_Small_US, Resistor_THT:R_Axial_DIN0204_L3.6mm_D1.6mm_P7.62mm_Horizontal, symbol Device:R_Small_US
- added R21: 1k, symbol Device:R_Small_US
- added RV4, RV5: R_Potentiometer_Trim_US, Potentiometer_THT:Potentiometer_Bourns_3296W_Vertical, symbol Device:R_Potentiometer_Trim_US
- added U4: LM358, Package_DIP:DIP-8_W7.62mm_Socket, symbol Amplifier_Operational:LM358
- added U5: TL494, Package_DIP:DIP-18_W7.62mm_Socket, symbol Regulator_Controller:TL494
Connections:
- net !PWM: no longer J3.3 (Pin_3), R9.1, U3.10 (E2)
- net +12V: now also C15.1, R20.1, U5.11 (C2), U5.12 (VCC)
- net +9V: now also C11.1, U4.8 (V+)
- net AUDIO: no longer C7.2, R12.1, R6.2, U2.7, U3.1 (1IN+)
- net FB: now also U5.2 (1IN-), U5.3 (FB)
- net GND: now also C11.2, C14.2, C15.2, J2.S, J4.2 (Pin_2), R13.2, R17.2, R19.2, R21.2, U4.4 (V-), U5.13 (OUTCTRL), U5.16 (2IN+), U5.4 (DTC), U5.7 (GND), U5.9 (E1)
- net PWM: no longer J3.1 (Pin_1), R8.2, U3.8 (C1)
- net SAWTOOTH: now also C14.1, U5.5 (CT)
- net VDC: now also U4.5 (+); no longer C10.1, R3.2, RV2.2, RV2.3
- net VDD: now also C10.1, R3.2, RV2.2, RV2.3, U4.3 (+)
- new net: C12.2, C13.1, R18.1, U4.6 (-)
- new net: R14.2, R15.1, U4.2 (-)
- new net: R15.2, RV4.1
- new net: R16.1, R17.1, RV4.2, RV4.3, U4.1
- new net: C12.1, R16.2
- new net: RV5.1, RV5.2, U5.6 (RT)
- new net: R13.1, RV5.3
- new net: C5.2, R14.1
- new net: C5.1, J2.R
- new net: U5.14 (REF), U5.15 (2IN-)
- new net !PWM_L: R9.1, U3.10 (E2)
- new net !PWM_R: J3.3 (Pin_3), J4.3 (Pin_3), R21.1, U5.10 (E2)
- new net AUDIO_L: C7.2, R12.1, R6.2, U2.7, U3.1 (1IN+)
- new net AUDIO_R: C13.2, R18.2, R19.1, U4.7, U5.1 (1IN+)
- new net PWM_L: J3.1 (Pin_1), J4.1 (Pin_1), R8.2, U3.8 (C1)
- new net PWM_R: R20.2, U5.8 (C1)
Other:
- note removed: "@Mundo Electronica"
- moved on the sheet: H1, H2, H3, H4, TP1, TP2, TP3, TP4, TP5, TP6, TP7, TP8
