File: PowerStage/PowerStage.kicad_pcb (KiCad board)
At the start: 2 copper layers, 41 parts, among them J1 Conn_01x02, J2 Conn_01x02, J3 Conn_01x03, Q1 IRFZ44N, Q2 IRFZ44N, Q3 IRFZ44N, Q4 IRFZ44N, U1 IR2110, U2 IR2110

Commit message: PCB desing init
Parts:
- added TP1: TestPoint, TestPoint:TestPoint_Keystone_5010-5014_Multipurpose, F.Cu at (200.9, 35.9)
- added TP2: TestPoint, TestPoint:TestPoint_Keystone_5010-5014_Multipurpose, F.Cu at (200.9, 41.0)
- added TP3: TestPoint, TestPoint:TestPoint_Keystone_5010-5014_Multipurpose, F.Cu at (200.9, 46.0)
- added TP4: TestPoint, TestPoint:TestPoint_Keystone_5010-5014_Multipurpose, F.Cu at (205.9, 35.9)
- added TP5: TestPoint, TestPoint:TestPoint_Keystone_5010-5014_Multipurpose, F.Cu at (205.9, 41.0)
- added TP6: TestPoint, TestPoint:TestPoint_Keystone_5010-5014_Multipurpose, F.Cu at (205.9, 46.0)
- added TP7: TestPoint, TestPoint:TestPoint_Keystone_5010-5014_Multipurpose, F.Cu at (211.0, 35.9)
- added TP8: TestPoint, TestPoint:TestPoint_Keystone_5010-5014_Multipurpose, F.Cu at (211.0, 41.0)
- added TP9: TestPoint, TestPoint:TestPoint_Keystone_5010-5014_Multipurpose, F.Cu at (211.0, 46.0)
- C11, C7: footprint Capacitor_THT:CP_Radial_D12.5mm_P5.00mm -> Capacitor_THT:C_Disc_D3.8mm_W2.6mm_P2.50mm
- moved L1 87.4 mm to (110.0, 83.0)
- moved R6 74.9 mm to (170.4, 52.0)
- moved C2 43.4 mm to (104.5, 50.5)
- moved L2 35.3 mm to (156.5, 83.5)
- moved C10 35.2 mm to (135.0, 50.5)
- moved C5 35.2 mm to (135.0, 37.5)
- moved C9 35.2 mm to (135.0, 44.0)
- moved Q1 35.2 mm to (156.4, 31.6)
- moved Q2 35.2 mm to (156.4, 37.5)
- moved Q3 35.2 mm to (156.4, 43.5)
- moved R1 35.2 mm to (166.7, 30.2)
- moved R3 35.2 mm to (166.7, 40.5)
- moved D1 35.2 mm to (141.1, 29.8)
- moved D2 35.2 mm to (141.1, 34.0)
- moved D3 35.2 mm to (141.1, 38.2)
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Connections:
- JP1 pad 2: +12V -> GND
- JP2 pad 2: +12V -> GND
- R5 pad 2: GND -> +12V
- R6 pad 2: GND -> +12V

Commit message: PCB design progress
Parts:
- !PWM  GND  PWM: renamed from J3
- GND  12V: renamed from J2
- moved JP2 89.4 mm to (84.5, 77.9)
- moved C1 69.4 mm to (85.3, 105.2)
- moved U1 34.7 mm to (99.8, 104.4), turned to 180 degrees
- moved C3 15.8 mm to (121.2, 107.1)
- moved L1 14.9 mm to (124.3, 87.0)
- moved !PWM  GND  PWM 4.75 mm to (75.0, 99.5), turned to 90 degrees
Routing:
- net PWM: track 0.00 -> 17.3 mm
- net !PWM: track 0.00 -> 17.2 mm

Commit message: Rev 1.0 Gerber
Parts:
- GND 12V: renamed from GND  12V
- GNDPWR: renamed from J1; footprint Connector_JST:JST_XH_B2B-XH-A_1x02_P2.50mm_Vertical -> Connector_JST:JST_VH_B2P-VH_1x02_P3.96mm_Vertical
- PWM GND !PWM: renamed from !PWM  GND  PWM
- moved H4 182.6 mm to (54.1, 128.3)
- moved H2 171.2 mm to (55.2, 78.7)
- moved R5 148.5 mm to (228.6, 94.6), turned to 180 degrees
- moved TP2 126.2 mm to (84.5, 89.5)
- moved TP1 122.1 mm to (88.9, 84.5)
- moved R2 116.2 mm to (85.7, 118.7)
- moved R6 112.8 mm to (64.8, 91.4)
- moved C9 110.6 mm to (229.8, 101.0)
- moved R1 109.3 mm to (85.1, 102.9)
- moved C10 108.4 mm to (234.9, 92.7)
- moved C11 107.0 mm to (182.9, 88.3), turned to 180 degrees
- moved D6 105.4 mm to (228.6, 109.9), turned to 180 degrees
- moved TP3 105.1 mm to (117.5, 109.9)
- moved D1 101.4 mm to (78.1, 109.2), turned to 180 degrees
- moved D5 96.1 mm to (210.2, 113.7), turned to 180 degrees
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- renumbered JP2 to ON/OFF
Connections:
- L1 pad 1: Net-(Q1-S) -> Net-(C4-Pad1)
- L1 pad 2: Net-(C4-Pad1) -> Net-(Q1-S)
Routing:
- net !PWM: track 17.2 -> 232.9 mm
- net PWM: track 17.3 -> 227.5 mm
- net Net-(Q1-S): track 0.00 -> 119.0 mm
- net Net-(Q3-S): track 0.00 -> 108.3 mm
- net Net-(C4-Pad1): track 0.00 -> 57.7 mm
- net Net-(D5-K): track 0.00 -> 55.3 mm
- net Net-(C4-Pad2): track 0.00 -> 48.0 mm
- net Net-(D4-K): track 0.00 -> 46.5 mm
- net Net-(D5-A): track 0.00 -> 44.6 mm
- net Net-(JP2-A): track 0.00 -> 43.2 mm
- net Net-(JP1-A): track 0.00 -> 37.9 mm
- net Net-(D4-A): track 0.00 -> 36.4 mm
- net Net-(D3-K): track 0.00 -> 35.6 mm
- net Net-(D3-A): track 0.00 -> 30.4 mm
- net Net-(D2-A): track 0.00 -> 30.1 mm
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- added copper zone on F.Cu, net +12V
- added copper zone on B.Cu, net GND
- added copper zone on B.Cu, net GNDPWR
- added copper zone on F.Cu, net VDC
Other:
- board outline added: 207 x 67.3 mm
- board text added: "."
- board text added: "Cutoff Frecuency"
- board text added: "FULL BRIDGE REV 1.0 VIVA MEXICO"
- board text added: "ON/OFF"
- board text added: "SOLDER = ON"
- board text added: "VDC 48V MAX"
- board text added: "VICTOR ROSALES CLASS D FULL BRIDGE AMPLIFIER"

Commit message: Revision 1.1 in progress
Parts:
- removed C4: 680nF, Capacitor_THT:C_Rect_L24.0mm_W8.3mm_P22.50mm_MKT
- removed GND 12V: Conn_01x02, Connector_JST:JST_XH_B2B-XH-A_1x02_P2.50mm_Vertical
- removed GNDPWR: Conn_01x02, Connector_JST:JST_VH_B2P-VH_1x02_P3.96mm_Vertical
- removed JP1, ON/OFF: SolderJumper_2_Open, Jumper:SolderJumper-2_P1.3mm_Open_Pad1.0x1.5mm
- removed PWM GND !PWM: Conn_01x03, Connector_JST:JST_XH_B3B-XH-A_1x03_P2.50mm_Vertical
- added C12: 100nF 1206, Capacitor_SMD:C_1206_3216Metric, F.Cu at (75.7, 81.8)
- added C13: 100nF-1206, Capacitor_SMD:C_1206_3216Metric, F.Cu at (75.4, 91.3)
- added J1: Conn_01x02, Connector_JST:JST_VH_B2P-VH_1x02_P3.96mm_Vertical, F.Cu at (121.3, 97.1)
- added J2: Conn_01x02, Connector_JST:JST_XH_B2B-XH-A_1x02_P2.50mm_Vertical, F.Cu at (108.7, 100.1)
- added J3: Conn_01x03, Connector_JST:JST_XH_B3B-XH-A_1x03_P2.50mm_Vertical, F.Cu at (108.7, 107.9)
- added SW1: K2-2235D-F1, lcsc_footprints:C108742_SW-TH_K2-2235D-F1, F.Cu at (75.5, 86.6)
- added SW2: K2-2235D-F1, lcsc_footprints:C108742_SW-TH_K2-2235D-F1, F.Cu at (76.0, 95.4)
- Q1, Q2, Q3, Q4: value IRFZ44N -> IRFB4227PBF; footprint Package_TO_SOT_THT:TO-220-3_Vertical -> lcsc_footprints:C2652_TO-220-3_L10_0-W4_5-P2_54-L
- R1, R2, R3, R4: footprint Resistor_THT:R_Axial_DIN0207_L6.3mm_D2.5mm_P7.62mm_Horizontal -> Resistor_SMD:R_1206_3216Metric
- R5, R6: value 10k -> 10k-1206; footprint Resistor_THT:R_Axial_DIN0207_L6.3mm_D2.5mm_P7.62mm_Horizontal -> Resistor_SMD:R_1206_3216Metric
- moved H3 180.2 mm to (78.6, 68.6)
- moved H1 172.5 mm to (78.6, 52.7)
- moved R5 146.9 mm to (82.2, 81.8), turned to 0 degrees
- moved U2 136.0 mm to (104.7, 79.9)
- moved C10 110.9 mm to (126.0, 71.7)
- moved C9 109.8 mm to (126.0, 65.1)
- moved R4 105.0 mm to (96.0, 110.9)
- moved R3 104.7 mm to (96.0, 106.8)
- moved Q4 104.5 mm to (88.5, 73.9), turned to 0 degrees
- moved D6 103.6 mm to (132.1, 72.1), turned to 0 degrees
- moved Q3 102.3 mm to (88.5, 66.8), turned to 0 degrees
- moved D5 90.5 mm to (132.1, 67.9), turned to 0 degrees
- moved D4 85.2 mm to (132.1, 63.6), turned to 0 degrees
- moved TP2 80.5 mm to (157.9, 56.6)
- moved C1 79.8 mm to (126.0, 52.0)
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Connections:
- C1 pad 1: GND -> +12V
- C1 pad 2: +12V -> GND
- C11 pad 2: GNDPWR -> GND
- C2 pad 2: GNDPWR -> GND
- C3 pad 2: GNDPWR -> GND
- C7 pad 2: GNDPWR -> GND
- C8 pad 2: GNDPWR -> GND
- Q1 pad 1: VDC -> Net-(D2-A)
- Q1 pad 2: Net-(D2-A) -> VDC
- Q2 pad 1: Net-(Q1-S) -> Net-(D3-A)
- Q2 pad 2: Net-(D3-A) -> Net-(Q1-S)
- Q2 pad 3: GNDPWR -> GND
- Q3 pad 1: VDC -> Net-(D4-A)
- Q3 pad 2: Net-(D4-A) -> VDC
- Q4 pad 1: Net-(Q3-S) -> Net-(D5-A)
- Q4 pad 2: Net-(D5-A) -> Net-(Q3-S)
- Q4 pad 3: GNDPWR -> GND
- R5 pad 1: Net-(JP1-A) -> Net-(U1-SD)
- R5 pad 2: +12V -> GND
- R6 pad 1: Net-(JP2-A) -> Net-(U2-SD)
- R6 pad 2: +12V -> GND
- TP4 pad 1: GNDPWR -> unconnected-(TP4-Pad1)
- TP8 pad 1: GNDPWR -> GND
- U1 pad 11: Net-(JP2-A) -> Net-(U1-SD)
- U1 pad 2: GNDPWR -> GND
- U2 pad 11: Net-(JP1-A) -> Net-(U2-SD)
- U2 pad 2: GNDPWR -> GND
Routing:
- net !PWM: track 232.9 -> 0.00 mm
- net PWM: track 227.5 -> 0.00 mm
- net Net-(Q1-S): track 119.0 -> 0.00 mm
- net Net-(Q3-S): track 108.3 -> 50.2 mm
- net Net-(C6-Pad1): track 57.7 -> 0.00 mm
- net Net-(D5-K): track 55.3 -> 0.00 mm
- net Net-(C6-Pad2): track 48.0 -> 0.00 mm
- net Net-(D4-K): track 46.5 -> 0.00 mm
- net Net-(D5-A): track 44.6 -> 0.00 mm
- net Net-(JP2-A): track 43.2 -> 0.00 mm
- net Net-(JP1-A): track 37.9 -> 0.00 mm
- net Net-(D4-A): track 36.4 -> 0.00 mm
- net Net-(D3-K): track 35.6 -> 0.00 mm
- net Net-(D3-A): track 30.4 -> 0.00 mm
- net Net-(D2-A): track 30.1 -> 0.00 mm
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- added copper zone on B.Cu, net (none)
- removed copper zone on F.Cu, net +12V
- removed copper zone on B.Cu, net GNDPWR
- removed copper zone on F.Cu, net VDC
Other:
- board outline removed
- copper layers 2 -> 4
- board text removed: "."
- board text removed: "Cutoff Frecuency"
- board text removed: "FULL BRIDGE REV 1.0 VIVA MEXICO"
- board text removed: "ON/OFF"
- board text removed: "SOLDER = ON"
- board text removed: "VDC 48V MAX"
- board text removed: "VICTOR ROSALES CLASS D FULL BRIDGE AMPLIFIER"

Commit message: Rev 1.1 progress
Parts:
- added C4: 100uF, Capacitor_THT:CP_Radial_D8.0mm_P3.80mm, F.Cu at (162.7, 77.5)
- C11, C7: footprint Capacitor_THT:C_Disc_D3.8mm_W2.6mm_P2.50mm -> Capacitor_SMD:C_1206_3216Metric
- L1, L2: value 47uH -> MDA1365-470M; footprint Inductor_SMD:L_12x12mm_H6mm -> lcsc_footprints:C2847587_IND-SMD_L13_5-W12_6_TMPA1265SP-100MN-D
- moved H3 101.5 mm to (176.5, 41.9)
- moved ON-OFF 100.8 mm to (175.3, 77.7)
- moved TP3 98.4 mm to (66.1, 97.2)
- moved TP7 98.4 mm to (76.2, 87.1)
- moved TP8 98.4 mm to (76.2, 92.1)
- moved TP9 98.4 mm to (76.2, 97.2)
- moved TP4 98.4 mm to (71.2, 87.1)
- moved TP5 98.4 mm to (71.2, 92.1)
- moved TP6 98.4 mm to (71.2, 97.2)
- moved C13 95.7 mm to (166.4, 61.6), turned to -90 degrees
- moved R6 94.1 mm to (175.3, 73.0)
- moved Gate-Q1 93.5 mm to (64.8, 43.2)
- moved Gate-Q2 83.3 mm to (77.5, 78.1)
- moved R3 79.2 mm to (154.9, 54.0), turned to 90 degrees
- moved D1 78.8 mm to (53.3, 49.5)
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- renumbered TP1 to Gate-Q1, TP2 to Gate-Q2, SW1 to ON-OFF, SW2 to ON-OFF
Connections:
- L1 pad 1: Net-(C6-Pad1) -> Net-(Q1-S)
- L1 pad 2: Net-(Q1-S) -> Net-(C6-Pad1)
- L2 pad 2: Net-(Q3-S) -> unconnected-(L2-Pad2)
- Q1 pad 1: Net-(D2-A) -> unconnected-(Q1-G-Pad1)

Commit message: Rev 1.1 progress pcb layout
Parts:
- GND  12V: renamed from J2
- GND | VDD: renamed from J1
- moved GND 99.8 mm to (163.2, 43.2)
- moved GATE-Q3 97.0 mm to (154.9, 43.2)
- moved GATE-Q4 70.7 mm to (146.1, 76.2)
- moved VS2-NL 60.0 mm to (126.4, 73.7)
- moved GATEQ2 54.3 mm to (71.8, 43.2)
- moved GND 54.0 mm to (78.7, 43.2)
- moved GND 36.8 mm to (105.4, 73.7)
- moved PWM-GND-!PWM 5.90 mm to (118.7, 73.1), turned to 180 degrees
- moved GND | VDD 3.99 mm to (136.5, 72.2), turned to -90 degrees
- moved GND  12V 3.35 mm to (97.8, 74.2)
- moved ON-OFF 0.86 mm to (175.3, 78.5)
- moved C11 0.63 mm to (149.2, 46.4)
- moved H4 0.63 mm to (153.7, 77.5)
- moved R6 0.63 mm to (175.3, 73.7)
- moved U2 0.63 mm to (179.1, 69.8)
- renumbered TP5 to GATE-Q3, TP7 to GATE-Q4, TP3 to GATEQ2, TP4 to GND, TP8 to GND, TP9 to GND, Gate-Q1 to GateQ1, J3 to PWM-GND-!PWM, Gate-Q2 to VS1-NL, TP6 to VS2-NL
Other:
- board text added: "36V-2A"
- board text added: "MAX"

Commit message: PCB layout progress
Parts:
- J1: renamed from GND | VDD
- J2: renamed from GND  12V
- moved C9 1.27 mm to (165.0, 56.5)
- moved C13 0.90 mm to (167.0, 62.2), turned to 180 degrees
- turned R3 to -90 degrees
- renumbered PWM-GND-!PWM to J3, ON-OFF to SW1, ON-OFF to SW2, GateQ1 to TP1, VS1-NL to TP2, GATEQ2 to TP3, GND to TP4, GATE-Q3 to TP5, VS2-NL to TP6, GATE-Q4 to TP7, GND to TP8, GND to TP9
Connections:
- L1 pad 2: Net-(C6-Pad1) -> Net-(C6-Pad2)
- L2 pad 1: Net-(C6-Pad2) -> Net-(C6-Pad1)
- L2 pad 2: unconnected-(L2-Pad2) -> Net-(Q3-S)
- LS1 pad 1: Net-(C6-Pad2) -> Net-(C6-Pad1)
- LS1 pad 2: Net-(C6-Pad1) -> Net-(C6-Pad2)
Routing:
- net Net-(Q3-S): track 50.2 -> 0.00 mm
- net Net-(D4-K): track 0.00 -> 29.0 mm
- net Net-(D4-A): track 0.00 -> 19.9 mm
- net (no net): track 14.2 -> 0.00 mm
- net +12V: track 10.8 -> 0.00 mm
- net GND: track 10.1 -> 6.07 mm, vias 0 -> 5
- removed copper zone on B.Cu, net (none)
Other:
- board outline added: 132.7 x 47.6 mm
- board text added: "Victor Almaraz Rosales Class D BTL Amplifier"

Commit message: PCB layout progress
Parts:
- C2: value 470uF -> 470uF 16V; footprint Capacitor_THT:CP_Radial_D12.5mm_P5.00mm -> lcsc_footprints:C3341_CAP-SMD_BD8_0-L8_3-W8_3-FD
- C3: value 470uf -> 470uF 16V; footprint Capacitor_THT:CP_Radial_D12.5mm_P5.00mm -> lcsc_footprints:C3341_CAP-SMD_BD8_0-L8_3-W8_3-FD
- moved C3 44.3 mm to (137.1, 45.3)
- moved C2 39.6 mm to (95.3, 45.4)
- moved C6 22.5 mm to (127.5, 48.2), turned to 180 degrees
- moved D5 10.2 mm to (159.4, 72.4), turned to 90 degrees
- turned R4 to -90 degrees
Routing:
- net GND: track 6.07 -> 7.42 mm, vias 5 -> 6
