File: PowerStage/PowerStage.kicad_pcb (KiCad board)
At the start: 4 copper layers, 132.7 x 47.6 mm, 52 parts, among them J1 Conn_01x02, J2 Conn_01x02, J3 Conn_01x03, Q1 IRFB4227PBF, Q2 IRFB4227PBF, Q3 IRFB4227PBF, Q4 IRFB4227PBF, SW1 K2-2235D-F1, SW2 K2-2235D-F1, U1 IR2110, U2 IR2110

Commit message: PCB lay progress
Parts:
- moved D1 0.41 mm to (53.8, 49.5)
- moved D6 0.36 mm to (169.2, 49.5)
Routing:
- net GND: track 7.42 -> 35.7 mm, vias 6 -> 20
- net Net-(U1-SD): track 0.00 -> 3.56 mm
- added copper zone on F.Cu, net +12V

Commit message: PCB layout complete rev 1.1
Parts:
- moved J3 2.42 mm to (116.7, 71.8), turned to -90 degrees
- moved C4 1.38 mm to (163.2, 78.7)
- moved H4 1.00 mm to (153.0, 76.7)
- moved C10 0.86 mm to (164.1, 67.9)
- moved SW1 0.43 mm to (57.8, 78.7)
- renumbered TP4 to GND, TP8 to GND, TP5 to GQ3, TP2 to SWN-1, TP7 to SWN-2
Connections:
- GND pad 1: unconnected-(TP4-Pad1) -> GND
- Q1 pad 1: unconnected-(Q1-G-Pad1) -> Net-(D2-A)
Routing:
- net PWM: track 0.00 -> 134.7 mm
- net !PWM: track 0.00 -> 126.2 mm
- net Net-(Q3-S): track 0.00 -> 64.0 mm
- net Net-(Q1-S): track 0.00 -> 56.1 mm
- net Net-(D3-K): track 0.00 -> 40.6 mm
- net Net-(D2-K): track 0.00 -> 36.5 mm
- net Net-(D1-K): track 0.00 -> 35.0 mm
- net Net-(D5-A): track 0.00 -> 32.1 mm
- net Net-(D3-A): track 0.00 -> 30.7 mm
- net Net-(D5-K): track 0.00 -> 26.9 mm
- net Net-(C6-Pad1): track 0.00 -> 25.5 mm
- net Net-(C6-Pad2): track 0.00 -> 25.1 mm
- net Net-(D2-A): track 0.00 -> 22.7 mm
- net Net-(D6-K): track 0.00 -> 21.8 mm
- net Net-(U2-SD): track 0.00 -> 19.2 mm
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- added copper zone on In2.Cu, net +12V
- added copper zone on In1.Cu, net GND
- added copper zone on F.Cu, net Net-(Q1-S)
- added copper zone on F.Cu, net Net-(Q3-S)
- added copper zone on F.Cu, net VDC
- removed copper zone on F.Cu, net +12V

Commit message: Silkscreen edit top
Parts:
- renumbered TP9 to GND, TP1 to GQ1, TP3 to GQ2, SWN-2 to GQ4, SW1 to ON<>OFF, SW2 to ON<>OFF, TP6 to SWN-2
Changed lines of the file:
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@@
 		(descr "Keystone THM Multipurpose Test Point 5010-5014, http://www.keyelco.com/product-pdf.cfm?p=1319")
 		(tags "Through Hole Mount Test Points")
-		(property "Reference" "SWN-2"
+		(property "Reference" "GQ4"
 			(at 0.635 -2.75 0)
 			(layer "F.SilkS")
@@
 		(descr "Keystone THM Multipurpose Test Point 5010-5014, http://www.keyelco.com/product-pdf.cfm?p=1319")
 		(tags "Through Hole Mount Test Points")
-		(property "Reference" "TP3"
+		(property "Reference" "GQ2"
 			(at 0 -2.75 0)
 			(layer "F.SilkS")
@@
 		(descr "Keystone THM Multipurpose Test Point 5010-5014, http://www.keyelco.com/product-pdf.cfm?p=1319")
 		(tags "Through Hole Mount Test Points")
-		(property "Reference" "TP1"
+		(property "Reference" "GQ1"
 			(at 0 -2.75 0)
 			(layer "F.SilkS")
@@
 		(descr "Keystone THM Multipurpose Test Point 5010-5014, http://www.keyelco.com/product-pdf.cfm?p=1319")
 		(tags "Through Hole Mount Test Points")
-		(property "Reference" "TP6"
+		(property "Reference" "SWN-2"
 			(at 0 -2.75 0)
 			(layer "F.SilkS")
@@
 		(layer "F.Cu")
 		(at 57.785 78.74)
-		(property "Reference" "SW1"
+		(property "Reference" "ON<>OFF"
 			(at 0 3.81 0)
 			(layer "F.SilkS")
@@
 		(descr "Keystone THM Multipurpose Test Point 5010-5014, http://www.keyelco.com/product-pdf.cfm?p=1319")
 		(tags "Through Hole Mount Test Points")
-		(property "Reference" "TP9"
+		(property "Reference" "GND"
 			(at 0 -2.75 0)
 			(layer "F.SilkS")
@@
 		(layer "F.Cu")
 		(at 175.26 78.535)
-		(property "Reference" "SW2"
+		(property "Reference" "ON<>OFF"
 			(at 0 3.605 0)
 			(layer "F.SilkS")

Commit message: Added graphics to silkscreen
Parts:
- added G***: LOGO, cat_4, B.Cu at (94.3, 59.2)
- added G***: LOGO, cat_4, B.Cu at (139.4, 59.6)
- added G***: LOGO, victor_logo_2, B.Cu at (116.7, 45.7)

Commit message: Rev 1.2
Parts:
- C2, C3: footprint lcsc_footprints:C3341_CAP-SMD_BD8_0-L8_3-W8_3-FD -> lcsc_footprints:C46550425_CAP-TH_BD10_0-P5_00-D0_6-FD-A
- C9: value 10uF -> 1uF
- GNDT1, GNDT2, GNDT3: renamed from GND; footprint TestPoint:TestPoint_Keystone_5010-5014_Multipurpose -> lcsc_footprints:C5277086_TEST-TH_BD2_54-P1_4_RED
- GQ1, GQ2, GQ3, GQ4: footprint TestPoint:TestPoint_Keystone_5010-5014_Multipurpose -> lcsc_footprints:C5277086_TEST-TH_BD2_54-P1_4_RED
- N1: renamed from SWN-1; footprint TestPoint:TestPoint_Keystone_5010-5014_Multipurpose -> lcsc_footprints:C5277086_TEST-TH_BD2_54-P1_4_RED
- N2: renamed from SWN-2; footprint TestPoint:TestPoint_Keystone_5010-5014_Multipurpose -> lcsc_footprints:C5277086_TEST-TH_BD2_54-P1_4_RED
- moved C2 1.13 mm to (94.6, 44.5)
- moved C3 1.12 mm to (137.8, 44.5)
- moved G*** 0.96 mm to (138.4, 59.6)
- moved G*** 0.31 mm to (94.6, 59.2)
- renumbered ON<>OFF to SW1, ON<>OFF to SW2
Routing:
- net GND: track 35.7 -> 7.42 mm, vias 20 -> 6
Other:
- board text added: "GND|12V"
- board text added: "GND|VDD"
- board text added: "ON<>OFF"
- board text added: "PWM|GND|!PWM"
