File: PowerStage/PowerStage.kicad_sch (KiCad schematic)
At the start: 52 parts, among them J1 Conn_01x02, J2 Conn_01x02, J3 Conn_01x03, Q1 IRFB4227PBF, Q2 IRFB4227PBF, Q3 IRFB4227PBF, Q4 IRFB4227PBF, SW1 K2-2235D-F1, SW2 K2-2235D-F1, U1 IR2110, U2 IR2110

Commit message: PCB layout complete rev 1.1
Connections:
- net GND: now also TP4.1
- net at Q1.1 (G): now also D2.2 (A), R1.2, TP1.1
Other:
- moved on the sheet: Q1, TP4
Changed lines of the file:
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@@
 	)
 	(junction
-		(at 154.686 32.258)
+		(at 100.838 64.77)
 		(diameter 0)
 		(color 0 0 0 0)
 	)
 	(junction
-		(at 165.1 44.196)
+		(at 154.686 32.258)
 		(diameter 0)
 		(color 0 0 0 0)
 	)
 	(junction
-		(at 88.646 44.704)
+		(at 165.1 44.196)
 		(diameter 0)
 		(color 0 0 0 0)
@@
 	)
 	(junction
+		(at 87.63 44.45)
+		(diameter 0)
+		(color 0 0 0 0)
+	)
+	(junction
 		(at 154.94 52.07)
 		(diameter 0)
@@
 	(wire
 		(pts
-			(xy 88.646 44.704) (xy 94.488 44.704)
-		)
-		(stroke
-			(width 0)
-			(type default)
-		)
-	)
-	(wire
-		(pts
 			(xy 129.286 32.258) (xy 134.874 32.258)
 		)
@@
 	(wire
 		(pts
+			(xy 95.25 64.77) (xy 100.838 64.77)
+		)
+		(stroke
+			(width 0)
+			(type default)
+		)
+	)
+	(wire
+		(pts
 			(xy 186.69 59.69) (xy 186.69 59.944)
 		)
@@
 	(wire
 		(pts
+			(xy 100.838 64.77) (xy 101.6 64.77)
+		)
+		(stroke
+			(width 0)
+			(type default)
+		)
+	)
+	(wire
+		(pts
 			(xy 67.056 58.674) (xy 68.326 58.674)
 		)
@@
 	(wire
 		(pts
-			(xy 101.6 49.784) (xy 100.838 49.784)
+			(xy 87.63 44.45) (xy 92.71 44.45)
+		)
+		(stroke
+			(width 0)
+			(type default)
+		)
+	)
+	(wire
+		(pts
+			(xy 101.6 49.784) (xy 100.33 49.53)
 		)
 		(stroke
@@
 	(wire
 		(pts
-			(xy 88.646 44.704) (xy 87.63 44.704)
+			(xy 88.646 44.704) (xy 87.63 44.45)
 		)
 		(stroke
@@
 	(wire
 		(pts
-			(xy 95.758 65.024) (xy 100.838 65.024)
-		)
-		(stroke
-			(width 0)
-			(type default)
-		)
-	)
-	(wire
-		(pts
 			(xy 166.37 56.388) (xy 162.306 56.388)
 		)
@@
 	(wire
 		(pts
-			(xy 78.74 44.704) (xy 80.01 44.704)
+			(xy 78.74 44.704) (xy 80.01 44.45)
 		)
 		(stroke
@@
 	(wire
 		(pts
-			(xy 100.838 33.528) (xy 100.838 39.624)
+			(xy 100.838 33.528) (xy 100.33 39.37)
 		)
 		(stroke
@@
 	(symbol
 		(lib_id "lcsc_imported:IRFB4227PBF")
-		(at 98.298 44.704 0)
+		(at 97.79 44.45 0)
 		(unit 1)
 		(exclude_from_sim no)
@@
 		(dnp no)
 		(property "Reference" "Q1"
-			(at 105.41 43.4339 0)
+			(at 104.902 43.1799 0)
 			(effects
 				(font
@@
 		)
 		(property "Value" "IRFB4227PBF"
-			(at 104.648 41.402 0)
+			(at 104.14 41.148 0)
 			(effects
 				(font
@@
 		)
 		(property "Footprint" "lcsc_footprints:C2652_TO-220-3_L10_0-W4_5-P2_54-L"
-			(at 98.298 54.864 0)
+			(at 97.79 54.61 0)
 			(effects
 				(font
@@
 		)
 		(property "Datasheet" "https://www.lcsc.com/datasheet/lcsc_datasheet_2304140030_Infineon-Technologies-IRFB4227PBF_C2652.pdf"
-			(at 96.012 44.577 0)
+			(at 95.504 44.323 0)
 			(effects
 				(font
@@
 		)
 		(property "Description" "IRFB4227PBF"
-			(at 98.298 44.704 0)
+			(at 97.79 44.45 0)
 			(effects
 				(font
@@
 		)
 		(property "LCSC" "C2652"
-			(at 98.298 44.704 0)
+			(at 97.79 44.45 0)
 			(effects
 				(font
@@
 		)
 		(property "Manufacturer" "Infineon(英飞凌)"
-			(at 98.298 44.704 0)
+			(at 97.79 44.45 0)
 			(effects
 				(font
@@
 	(symbol
 		(lib_id "Connector:TestPoint")
-		(at 95.758 65.024 90)
+		(at 95.25 64.77 90)
 		(unit 1)
 		(exclude_from_sim no)
@@
 		(dnp no)
 		(property "Reference" "TP4"
-			(at 94.234 62.738 90)
+			(at 93.726 62.484 90)
 			(effects
 				(font
@@
 		)
 		(property "Value" "TestPoint"
-			(at 97.282 67.056 90)
+			(at 96.774 66.802 90)
 			(effects
 				(font
@@
 		)
 		(property "Footprint" "TestPoint:TestPoint_Keystone_5010-5014_Multipurpose"
-			(at 95.758 59.944 0)
+			(at 95.25 59.69 0)
 			(effects
 				(font
@@
 		)
 		(property "Datasheet" "~"
-			(at 95.758 59.944 0)
+			(at 95.25 59.69 0)
 			(effects
 				(font
@@
 		)
 		(property "Description" "test point"
-			(at 95.758 65.024 0)
+			(at 95.25 64.77 0)
 			(effects
 				(font
@@
 	(symbol
 		(lib_id "Diode:1N5819")
-		(at 83.82 44.704 0)
+		(at 83.82 44.45 0)
 		(unit 1)
 		(exclude_from_sim no)
@@
 		(dnp no)
 		(property "Reference" "D2"
-			(at 84.074 47.244 0)
+			(at 84.074 46.99 0)
 			(effects
 				(font
@@
 		)
 		(property "Value" "1N5819"
-			(at 83.82 49.276 0)
+			(at 83.82 49.022 0)
 			(effects
 				(font
@@
 		)
 		(property "Footprint" "Diode_THT:D_DO-41_SOD81_P10.16mm_Horizontal"
-			(at 83.82 49.149 0)
+			(at 83.82 48.895 0)
 			(effects
 				(font
@@
 		)
 		(property "Datasheet" "http://www.vishay.com/docs/88525/1n5817.pdf"
-			(at 83.82 44.704 0)
+			(at 83.82 44.45 0)
 			(effects
 				(font
@@
 		)
 		(property "Description" "40V 1A Schottky Barrier Rectifier Diode, DO-41"
-			(at 83.82 44.704 0)
+			(at 83.82 44.45 0)
 			(effects
 				(font

Commit message: Rev 1.2
Parts:
- C1, C10, C5: LCSC (none) -> C330941
- C11, C12, C13, C7: LCSC (none) -> C24497
- C2, C3: footprint lcsc_footprints:C3341_CAP-SMD_BD8_0-L8_3-W8_3-FD -> lcsc_footprints:C46550425_CAP-TH_BD10_0-P5_00-D0_6-FD-A; LCSC C3341 -> C2837182
- C4, C8: footprint Capacitor_THT:CP_Radial_D8.0mm_P3.80mm -> Capacitor_THT:CP_Radial_D8.0mm_P3.50mm; LCSC (none) -> C1669449
- C6, J1, J2, J3, LS1, U1, U2: now left out of the parts list
- C9: value 10uF -> 1uF; LCSC (none) -> C330941
- D1, D2, D3, D4, D5, D6: LCSC (none) -> C16588
- R1, R2, R3, R4: LCSC (none) -> C17903
- R5, R6: LCSC (none) -> C17902
- TP1, TP2, TP3, TP4, TP5, TP6, TP7, TP8, TP9: footprint TestPoint:TestPoint_Keystone_5010-5014_Multipurpose -> lcsc_footprints:C5277086_TEST-TH_BD2_54-P1_4_RED; LCSC (none) -> C5277086
